Commit message: modified z1_gripper urdf with removing evaluation string

File: arm_sim_pybullet/z1_description/z1_gripper.urdf (robot description, URDF)
Before this commit: robot z1_description, 10 links, 9 joints
Links:
- link link00: geometry collision cylinder length=0.051 radius=0.0325; visual mesh filename=package://z1_description/meshes/visual/z1_Link00.dae scale=1 1 1
- link link02: geometry collision cylinder length=0.051 radius=0.0325; collision cylinder length=0.102 radius=0.0325
- link link03: geometry collision cylinder length=0.059 radius=0.0325; collision cylinder length=0.116 radius=0.02
- link link04: geometry collision cylinder length=0.067 radius=0.0325; visual mesh filename=package://z1_description/meshes/visual/z1_Link04.dae scale=1 1 1
- link link06: geometry collision cylinder length=0.051 radius=0.0325; visual mesh filename=package://z1_description/meshes/visual/z1_Link06.dae scale=1 1 1
Joints:
- joint joint1: limit lower=${-PI*150/180} upper=${PI*150/180} effort=30.0 velocity=3.1415 -> lower=-2.6179938779914944 upper=2.6179938779914944 effort=30.0 velocity=3.1415
- joint joint2: limit lower=0.0 upper=${PI*170/180} effort=60.0 velocity=3.1415 -> lower=0.0 upper=2.9670597283903604 effort=60.0 velocity=3.1415
- joint joint3: limit lower=${-PI*165/180} upper=0.0 effort=30.0 velocity=3.1415 -> lower=-2.8797932657906435 upper=0.0 effort=30.0 velocity=3.1415
- joint joint4: limit lower=${-PI*87/180} upper=${PI*87/180} effort=30.0 velocity=3.1415 -> lower=-1.5184364492350666 upper=1.5184364492350666 effort=30.0 velocity=3.1415
- joint joint5: limit lower=${-PI*77/180} upper=${PI*77/180} effort=30.0 velocity=3.1415 -> lower=-1.3439035240356338 upper=1.3439035240356338 effort=30.0 velocity=3.1415
- joint joint6: limit lower=${-PI*160/180} upper=${PI*160/180} effort=30.0 velocity=3.1415 -> lower=-2.792526803190927 upper=2.792526803190927 effort=30.0 velocity=3.1415
- joint jointGripper: limit lower=${-PI*90/180} upper=0.0 effort=30.0 velocity=3.1415 -> lower=-1.5707963267948966 upper=0.0 effort=30.0 velocity=3.1415
